Commit message: Adds tars_control_lib_py; Updates readmes.

File: tars_robot/tars_description/urdf/tars.xacro (robot description, xacro)
@@ -4,11 +4,11 @@
   <!-- Constants for robot dimensions -->
   <xacro:property name="PI" value="3.1415926535897931"/>
-  <xacro:property name="width" value="0.2" /> <!-- Square dimensions (widthxwidth) of beams -->
-  <xacro:property name="depth" value="0.1" /> <!-- Square dimensions (widthxwidth) of beams -->
+  <xacro:property name="width" value="0.33" /> <!-- Square dimensions (widthxwidth) of beams -->
+  <xacro:property name="depth" value="0.2" /> <!-- Square dimensions (widthxwidth) of beams -->
   <xacro:property name="height1" value="2" /> <!-- Link 1 -->
   <xacro:property name="height2" value="2" /> <!-- Link 2 -->
   <xacro:property name="height3" value="2" /> <!-- Link 3 -->
   <xacro:property name="height4" value="2" /> <!-- Link 4 -->
-  <xacro:property name="segmentmass" value="5" /> <!-- Link Mass -->
+  <xacro:property name="segmentmass" value="30" /> <!-- Link Mass -->
   <xacro:property name="camera_link" value="0.05" /> <!-- Size of square 'camera' box -->
   <xacro:property name="axel_offset" value="0.05" /> <!-- Space btw top of beam and the each joint -->
@@ -74,5 +74,5 @@
     <actuator name="motor1">
       <hardwareInterface>EffortJointInterface</hardwareInterface>
-      <mechanicalReduction>1</mechanicalReduction>
+      <mechanicalReduction>100</mechanicalReduction>
     </actuator>
   </transmission>
@@ -84,5 +84,5 @@
     <actuator name="motor2">
       <hardwareInterface>EffortJointInterface</hardwareInterface>
-      <mechanicalReduction>1</mechanicalReduction>
+      <mechanicalReduction>100</mechanicalReduction>
     </actuator>
   </transmission>
@@ -94,5 +94,5 @@
     <actuator name="motor3">
       <hardwareInterface>EffortJointInterface</hardwareInterface>
-      <mechanicalReduction>1</mechanicalReduction>
+      <mechanicalReduction>100</mechanicalReduction>
     </actuator>
   </transmission>

Commit message: Modifes TARS robot to have joint above center; Adds acceleration, velocity, and effort limits.

File: tars_robot/tars_description/urdf/tars.xacro (robot description, xacro)
@@ -10,4 +10,5 @@
   <xacro:property name="height3" value="2" /> <!-- Link 3 -->
   <xacro:property name="height4" value="2" /> <!-- Link 4 -->
+  <xacro:property name="motor_offset" value="-0.25" /> <!-- Link 4 -->
   <xacro:property name="segmentmass" value="30" /> <!-- Link Mass -->
   <xacro:property name="camera_link" value="0.05" /> <!-- Size of square 'camera' box -->
@@ -20,5 +21,5 @@
     <link name="${name}">
       <collision>
-        <origin xyz="0 0 ${offset}" rpy="0 0 0"/>
+        <origin xyz="0 0 ${offset + motor_offset}" rpy="0 0 0"/>
         <geometry>
     <box size="${depth} ${width} ${height}"/>
@@ -26,5 +27,5 @@
       </collision>
       <visual>
-        <origin xyz="0 0 ${offset}" rpy="0 0 0"/>
+        <origin xyz="0 0 ${offset + motor_offset}" rpy="0 0 0"/>
         <geometry>
     <box size="${depth} ${width} ${height}"/>
@@ -51,5 +52,6 @@
     <origin xyz="0 ${width} 0" rpy="0 0 0"/>
     <axis xyz="0 1 0"/>
-    <dynamics damping="0.0"/>
+    <dynamics damping="0.7"/>
+    <limit velocity="1" effort="100.0"/>
   </joint>
   <joint name="joint2" type="continuous">
@@ -58,5 +60,6 @@
     <origin xyz="0 ${width} 0" rpy="0 0 0"/>
     <axis xyz="0 1 0"/>
-    <dynamics damping="0.0"/>
+    <dynamics damping="0.7"/>
+    <limit velocity="1" effort="100.0"/>
   </joint>
   <joint name="joint3" type="continuous">
@@ -65,5 +68,6 @@
     <origin xyz="0 ${width} 0" rpy="0 0 0"/>
     <axis xyz="0 1 0"/>
-    <dynamics damping="0.0"/>
+    <dynamics damping="0.7"/>
+    <limit velocity="1" effort="100.0"/>
   </joint>
   <transmission name="tran1">

Commit message: Updates max effort to allow robot to stand when on ground.

File: tars_robot/tars_description/urdf/tars.xacro (robot description, xacro)
@@ -53,5 +53,5 @@
     <axis xyz="0 1 0"/>
     <dynamics damping="0.7"/>
-    <limit velocity="1" effort="100.0"/>
+    <limit velocity="1" effort="1000.0"/>
   </joint>
   <joint name="joint2" type="continuous">
@@ -61,5 +61,5 @@
     <axis xyz="0 1 0"/>
     <dynamics damping="0.7"/>
-    <limit velocity="1" effort="100.0"/>
+    <limit velocity="1" effort="1000.0"/>
   </joint>
   <joint name="joint3" type="continuous">
@@ -69,5 +69,5 @@
     <axis xyz="0 1 0"/>
     <dynamics damping="0.7"/>
-    <limit velocity="1" effort="100.0"/>
+    <limit velocity="1" effort="1000.0"/>
   </joint>
   <transmission name="tran1">
@@ -78,5 +78,5 @@
     <actuator name="motor1">
       <hardwareInterface>EffortJointInterface</hardwareInterface>
-      <mechanicalReduction>100</mechanicalReduction>
+      <mechanicalReduction>1</mechanicalReduction>
     </actuator>
   </transmission>
@@ -88,5 +88,5 @@
     <actuator name="motor2">
       <hardwareInterface>EffortJointInterface</hardwareInterface>
-      <mechanicalReduction>100</mechanicalReduction>
+      <mechanicalReduction>1</mechanicalReduction>
     </actuator>
   </transmission>
@@ -98,5 +98,5 @@
     <actuator name="motor3">
       <hardwareInterface>EffortJointInterface</hardwareInterface>
-      <mechanicalReduction>100</mechanicalReduction>
+      <mechanicalReduction>1</mechanicalReduction>
     </actuator>
   </transmission>
